Commit message: playing around

File: misc/urdf/a300.urdf (robot description, URDF)
Before this commit: robot racer, 6 links, 5 joints
Links:
- link base_link: geometry collision cylinder length=.025 radius=.06; visual cylinder length=0.06 radius=0.015
- link prop0_link: geometry visual mesh filename=./mesh/a300/prop.dae scale=0.4 0.4 0.4
- link prop1_link: geometry visual mesh filename=./mesh/a300/prop.dae scale=0.4 0.4 0.4
- link prop2_link: geometry visual mesh filename=./mesh/a300/prop.dae scale=0.4 0.4 0.4
- link prop3_link: geometry visual mesh filename=./mesh/a300/prop.dae scale=0.4 0.4 0.4

Commit message: added px4 ctbr controller

File: misc/urdf/a300.urdf (robot description, URDF)
Before this commit: robot racer, 6 links, 5 joints
Links:
- link base_link: mass 0.830 -> 1.21
