Commit message: It works!! Desc: - Two agents cooperate to drive the cg of a rod to a target position - Single rotor thrust as control mode - No domain rand, no action delay, perfect state estimation (fixthese later) - Training time around 50 min

File: misc/urdf/bros300.urdf (robot description, URDF)
Before this commit: robot bros300, 26 links, 25 joints
Links:
- removed link segment_10_cylinder
- removed link segment_10_sphere
- removed link segment_6_cylinder
- removed link segment_6_sphere
- removed link segment_7_cylinder
- removed link segment_7_sphere
- removed link segment_8_cylinder
- removed link segment_8_sphere
- removed link segment_9_cylinder
- removed link segment_9_sphere
- link base_link: geometry collision box size=.16 .16 .05; collision cylinder length=0.06 radius=0.015
- link segment_1_cylinder: mass 0.0001 -> 0.002
- link segment_1_sphere: mass 1e-04 -> 0.002; geometry visual sphere radius=0.005
- link segment_2_cylinder: mass 0.0001 -> 0.002
- link segment_2_sphere: mass 1e-04 -> 0.002; geometry visual sphere radius=0.005
- link segment_3_cylinder: mass 0.0001 -> 0.002
- link segment_3_sphere: mass 1e-04 -> 0.002; geometry visual sphere radius=0.005
- link segment_4_cylinder: mass 0.0001 -> 0.002
- link segment_4_sphere: mass 1e-04 -> 0.002; geometry visual sphere radius=0.005
- link segment_5_cylinder: mass 0.0001 -> 0.002
- link segment_5_sphere: mass 1e-04 -> 0.002; geometry visual sphere radius=0.005
Joints:
- removed joint segment_10_sphere_to_cylinder
- removed joint segment_5_cylinder_to_segment_6_sphere
- removed joint segment_6_cylinder_to_segment_7_sphere
- removed joint segment_6_sphere_to_cylinder
- removed joint segment_7_cylinder_to_segment_8_sphere
- removed joint segment_7_sphere_to_cylinder
- removed joint segment_8_cylinder_to_segment_9_sphere
- removed joint segment_8_sphere_to_cylinder
- removed joint segment_9_cylinder_to_segment_10_sphere
- removed joint segment_9_sphere_to_cylinder
